File: lnchpd-kicad/lnchpd-kicad.kicad_pcb (KiCad board)
At the start: 2 copper layers, 57 x 62.1 mm, 7 parts, among them SW1 SW_Push, SW2 SW_Push, SW3 SW_Push, SW4 SW_Push, SW5 SW_Push, SW6 SW_Push

Commit message: updated the pcb with 2 buttons, updated gerber and drill files.
Parts:
- added SW7: SW_Push, Button_Switch_THT:SW_NKK_GW12LJP, F.Cu at (138.0, 123.5)
- added SW8: SW_Push, Button_Switch_THT:SW_NKK_GW12LJP, F.Cu at (138.0, 130.5)
Connections:
- A1 pad 10: unconnected-(A1-GPIO7-Pad10) -> Net-(A1-GPIO7)
- A1 pad 9: unconnected-(A1-GPIO6-Pad9) -> Net-(A1-GPIO6)
Routing:
- net Net-(A1-GND-Pad13): track 189.5 -> 224.2 mm
- net Net-(A1-GPIO7): track 0.00 -> 29.8 mm
- net Net-(A1-GPIO6): track 0.00 -> 24.8 mm
