File: lnchpd-kicad/lnchpd-kicad.kicad_sch (KiCad schematic)
At the start: 7 parts, among them SW1 SW_Push, SW2 SW_Push, SW3 SW_Push, SW4 SW_Push, SW5 SW_Push, SW6 SW_Push

Commit message: updated the pcb with 2 buttons, updated gerber and drill files.
Parts:
- added SW7, SW8: SW_Push, Button_Switch_THT:SW_NKK_GW12LJP, symbol Switch:SW_Push
Connections:
- net at A1.13 (GND), A1.18 (GND), A1.23 (GND)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: now also SW7.2, SW8.2
- net at A1.10 (GPIO7): now also SW8.1
- net at A1.9 (GPIO6): now also SW7.1
